Commit message: updated 5/19

File: template_project/kuka_iiwa.urdf (robot description, URDF)
Before this commit: robot kuka_iiwa, 12 links, 11 joints
Links:
- added link leftfinger, mass 0.1; visual box size=0.03 .02 0.1; visual mesh filename=../../../model/iiwa7/meshes/finger.obj
- added link lower_leftfinger, mass 0.1; visual box size=0.03 .02 0.1; visual mesh filename=../../../model/iiwa7/meshes/finger.obj
- added link lower_rightfinger, mass 0.1; visual box size=0.03 .02 0.1; visual mesh filename=../../../model/iiwa7/meshes/finger.obj
- added link rightfinger, mass 0.1; visual box size=0.03 .02 0.1; visual mesh filename=../../../model/iiwa7/meshes/finger.obj
- link link6: geometry visual mesh filename=../../../model/iiwa7/meshes/hand.obj scale=1 1 1; visual mesh filename=../../../model/iiwa7/meshes/link6.obj scale=1 1 1
Joints:
- added joint finger_joint1: type prismatic, parent link6, child leftfinger, origin xyz=-0.015 0.04 0.09 rpy=0 0 1.570796327, axis 0 1 0, limit lower=0.0 upper=0.04 effort=20 velocity=0.2
- added joint finger_joint2: type prismatic, parent link6, child rightfinger, origin xyz=0.015 0.04 0.09 rpy=0 0 -1.570796327, axis 0 1 0, limit lower=0.0 upper=0.04 effort=20 velocity=0.2
- added joint finger_joint3: type prismatic, parent link6, child lower_leftfinger, origin xyz=-0.015 -0.065 0.09 rpy=0 0 1.570796327, axis 1 0 0, limit lower=0.0 upper=0.04 effort=20 velocity=0.2
- added joint finger_joint4: type prismatic, parent link6, child lower_rightfinger, origin xyz=0.015 -0.065 0.09 rpy=0 0 -1.570796327, axis 1 0 0, limit lower=0.0 upper=0.04 effort=20 velocity=0.2
