Commit message: world integrated into panda gripper example

File: panda_gripper_example/panda_arm.urdf (robot description, URDF)
Before this commit: robot panda_arm, 8 links, 7 joints
Links:
- removed link link0
- added link base_link, mass 64.6; visual mesh filename=../../../model/mmp_panda/meshes/panda_BaseCombo.obj
- added link base_x, mass 0.001
- added link base_y, mass 0.001
- added link ground_link, mass 0.001
Joints:
- added joint base_prismatic_x: type prismatic, parent ground_link, child base_x, origin xyz=0 0 0 rpy=0 0 0, axis 1 0 0, limit lower=-2.8973 upper=2.9873 effort=87 velocity=2.1750
- added joint base_prismatic_y: type prismatic, parent base_x, child base_y, origin xyz=0 0 0 rpy=0 0 0, axis 0 1 0, limit lower=-2.8973 upper=2.9873 effort=87 velocity=2.1750
- added joint base_revolute: type revolute, parent base_y, child base_link, origin xyz=0 0 0.0 rpy=0 0 0, axis 0 0 1, limit lower=-2.8973 upper=2.8973 effort=87 velocity=2.1750
- joint joint1: parent link0 -> base_link

File: panda_gripper_example/panda_arm_hand.urdf (robot description, URDF)
Before this commit: robot panda_arm_hand, 10 links, 9 joints
Links:
- removed link link0
- added link base_link, mass 64.6; visual mesh filename=../../../model/mmp_panda/meshes/panda_BaseCombo.obj
- added link base_x, mass 0.001
- added link base_y, mass 0.001
- added link ground_link, mass 0.001
Joints:
- added joint base_prismatic_x: type prismatic, parent ground_link, child base_x, origin xyz=0 0 0 rpy=0 0 0, axis 1 0 0, limit lower=-2.8973 upper=2.9873 effort=87 velocity=2.1750
- added joint base_prismatic_y: type prismatic, parent base_x, child base_y, origin xyz=0 0 0 rpy=0 0 0, axis 0 1 0, limit lower=-2.8973 upper=2.9873 effort=87 velocity=2.1750
- added joint base_revolute: type revolute, parent base_y, child base_link, origin xyz=0 0 0.0 rpy=0 0 0, axis 0 0 1, limit lower=-2.8973 upper=2.8973 effort=87 velocity=2.1750
- joint joint1: parent link0 -> base_link

Commit message: ball not flying well idk

File: panda_gripper_example/panda_arm.urdf (robot description, URDF)
Before this commit: robot panda_arm, 11 links, 10 joints
Links:
- link base_link: geometry visual mesh filename=../../../model/iiwa7/meshes/kuka_mobile_base.obj

File: panda_gripper_example/panda_arm_hand.urdf (robot description, URDF)
Before this commit: robot panda_arm_hand, 15 links, 14 joints
Links:
- link base_link: geometry visual mesh filename=../../../model/iiwa7/meshes/kuka_mobile_base.obj
