Commit message: attempt at grasping ball

File: panda_gripper_example/panda_arm_hand.urdf (robot description, URDF)
Before this commit: robot panda_arm_hand, 13 links, 12 joints
Links:
- link leftfinger: geometry collision box size=0.2 .02 0.3; visual mesh filename=../../../model/panda/meshes/visual/finger.obj
- link rightfinger: geometry collision box size=0.2 .02 0.3; visual mesh filename=../../../model/panda/meshes/visual/finger.obj

Commit message: "arm flailing"

File: panda_gripper_example/panda_arm_hand.urdf (robot description, URDF)
Before this commit: robot panda_arm_hand, 13 links, 12 joints
Links:
- link leftfinger: geometry collision box size=0.2 .02 0.3; visual box size=0.2 .02 0.3
- link rightfinger: geometry collision box size=0.2 .02 0.3; visual box size=0.2 .02 0.3

Commit message: "hovering above ball"

File: panda_gripper_example/panda_arm_hand.urdf (robot description, URDF)
Before this commit: robot panda_arm_hand, 13 links, 12 joints
Links:
- link leftfinger: geometry collision box size=0.2 .02 0.2; visual box size=0.2 .02 0.2
- link rightfinger: geometry collision box size=0.2 .02 0.2; visual box size=0.2 .02 0.2

Commit message: "picking up ball"

File: panda_gripper_example/panda_arm_hand.urdf (robot description, URDF)
Before this commit: robot panda_arm_hand, 13 links, 12 joints
Links:
- link leftfinger: mass 0.1 -> .75
- link rightfinger: mass 0.1 -> 0.75

Commit message: "integrated with keypress base movement"

File: panda_gripper_example/panda_arm_hand.urdf (robot description, URDF)
Before this commit: robot panda_arm_hand, 13 links, 12 joints
Links:
- link leftfinger: geometry collision box size=0.2 .02 0.2; visual mesh filename=../../../model/panda/meshes/visual/finger.obj scale=2 2 2
- link rightfinger: geometry collision box size=0.2 .02 0.2; visual mesh filename=../../../model/panda/meshes/visual/finger.obj scale=2 2 2

Commit message: adjusted 2 fingers

File: panda_gripper_example/panda_arm_hand.urdf (robot description, URDF)
Before this commit: robot panda_arm_hand, 13 links, 12 joints
Links:
- link leftfinger: geometry collision box size=0.1 .02 0.2; visual box size=0.1 .02 0.2
- link rightfinger: geometry collision box size=0.1 .02 0.2; visual box size=0.1 .02 0.2
Joints:
- joint finger_joint1: origin xyz=0 0 0.1654 rpy=0 0 -0.78539816339 -> xyz=0 .08 0.1654 rpy=0 0 -0.98539816339
- joint finger_joint2: origin xyz=0 0 0.1654 rpy=0 0 -0.78539816339 -> xyz=0 .08 0.1654 rpy=0 0 -0.58539816339

Commit message: yeet the ball

File: panda_gripper_example/panda_arm_hand.urdf (robot description, URDF)
Before this commit: robot panda_arm_hand, 13 links, 12 joints
Links:
- added link leftfinger_bottom, mass .75; collision box size=0.1 .02 0.2; visual box size=0.1 .02 0.2
- added link rightfinger_bottom, mass 0.75; collision box size=0.1 .02 0.2; visual box size=0.1 .02 0.2
Joints:
- added joint finger_joint3: type prismatic, parent link7, child leftfinger_bottom, origin xyz=0.02 -.03 0.1654 rpy=0 0 -0.48539816339, axis 0 1 0, limit lower=0.0 upper=0.04 effort=20 velocity=0.2
- added joint finger_joint4: type prismatic, parent link7, child rightfinger_bottom, origin xyz=.06 -.03 0.1654 rpy=0 0 -1.08539816339, axis 0 1 0, limit lower=0.0 upper=0.04 effort=20 velocity=0.2
- joint finger_joint1: origin xyz=0 .08 0.1654 rpy=0 0 -0.98539816339 -> xyz=-.02 .03 0.1654 rpy=0 0 -1.08539816339
- joint finger_joint2: origin xyz=0 .08 0.1654 rpy=0 0 -0.58539816339 -> xyz=.02 .03 0.1654 rpy=0 0 -0.48539816339

Commit message: gripper orientation fixed

File: panda_gripper_example/panda_arm_hand.urdf (robot description, URDF)
Before this commit: robot panda_arm_hand, 15 links, 14 joints
Joints:
- joint finger_joint1: origin xyz=-.02 .03 0.1654 rpy=0 0 -1.08539816339 -> xyz=0 0 0.1654 rpy=0 0 -0.78539816339
- joint finger_joint2: origin xyz=.02 .03 0.1654 rpy=0 0 -0.48539816339 -> xyz=0 0 0.1654 rpy=0 0 -0.78539816339
- joint finger_joint3: axis 0 1 0 -> 1 0 0; origin xyz=0.02 -.03 0.1654 rpy=0 0 -0.48539816339 -> xyz=0 0 0.1654 rpy=0 0 -0.78539816339
- joint finger_joint4: axis 0 1 0 -> 1 0 0; origin xyz=.06 -.03 0.1654 rpy=0 0 -1.08539816339 -> xyz=0 0 0.1654 rpy=0 0 -0.78539816339

Commit message: working bowl

File: panda_gripper_example/panda_arm_hand.urdf (robot description, URDF)
Before this commit: robot panda_arm_hand, 15 links, 14 joints
Links:
- link leftfinger: mass .75 -> .25
- link leftfinger_bottom: mass .75 -> .25
- link rightfinger: mass 0.75 -> 0.25
- link rightfinger_bottom: mass 0.75 -> 0.25

Commit message: edited grippers and world

File: panda_gripper_example/panda_arm_hand.urdf (robot description, URDF)
Before this commit: robot panda_arm_hand, 15 links, 14 joints
Links:
- link leftfinger: geometry collision box size=0.1 .02 0.2; visual mesh filename=../../../model/panda/meshes/visual/gripper_new.obj scale=1 1 1
- link leftfinger_bottom: geometry collision box size=0.1 .02 0.2; visual mesh filename=../../../model/panda/meshes/visual/gripper_new.obj scale=1 1 1
- link link7: geometry visual mesh filename=../../../model/panda/meshes/visual/joint7_sphere.obj scale=3 3 2; visual mesh filename=../../../model/panda/meshes/visual/link7.obj
- link rightfinger: geometry collision box size=0.1 .02 0.2; visual mesh filename=../../../model/panda/meshes/visual/gripper_new.obj scale=1 1 1
- link rightfinger_bottom: geometry collision box size=0.1 .02 0.2; visual mesh filename=../../../model/panda/meshes/visual/gripper_new.obj scale=1 1 1
